File: ossc_board.kicad_pcb (KiCad board)
At the start: 2 copper layers, 124.6 x 68.7 mm, 226 parts, among them J1 VGA, J2 3XRCA_CONN, J3 SCART-F, J4 HDMI_CONN, J5 5VDC_IN, J6 SJ1-3533NG, J7 SJ1-3533NG, P1 JTAG_CONN, P3 mSD_CONN, Q1 BC847, Q2 BC857, SW1 SPST, SW2 SW_PUSH, SW3 SW_PUSH, SW4 DPDT, U1 TVP7002PZP, U10 S25FL216K, U11 IRM-V538/TR1, U12 TLV70012, U13 TLV70025, U14 TLV70012, U15 TLV70018, U16 TLV70018, U17 THS7353, U2 EP4CE15E22, U3 IT6613, U4 SN74LVC2G17, U5 AP7361C, U6 TLV70033, U7 NCP703SN19T1G, U8 PCM1862, U9 TLV70019, Y1 ACHL-27MHZ-EK, Y2 24.576MHz

Commit message: finalize pcb v1.6
Parts:
- removed C117, C122: 10u, custom_components:SM0603_Capa_libcms
- added R47: 100k, custom_components:SM0603_Resistor_libcms, B.Cu at (126.2, 33.8)
- added R48: 100k, custom_components:SM0603_Resistor_libcms, B.Cu at (124.0, 33.8)
- added R49: 100k, custom_components:SM0603_Resistor_libcms, B.Cu at (122.6, 70.9)
- added R50: 100k, custom_components:SM0603_Resistor_libcms, B.Cu at (120.2, 70.9)
- added R51: 100k, custom_components:SM0603_Resistor_libcms, B.Cu at (120.2, 74.4)
- added R52: 100k, custom_components:SM0603_Resistor_libcms, B.Cu at (120.2, 66.6)
- C111, C112: value 32p -> 30p; moved to B.Cu
- C113, C114, C115, C116, C118, C121, C123, C125: moved to B.Cu
- moved C121 63.8 mm to (115.2, 65.9), turned to 180 degrees
- moved C123 61.6 mm to (115.2, 73.9)
- moved C116 54.5 mm to (115.2, 67.6), turned to 180 degrees
- moved C118 52.2 mm to (106.2, 67.2), turned to 180 degrees
- moved C114 50.4 mm to (111.8, 66.0), turned to 90 degrees
- moved C125 50.1 mm to (115.2, 72.1)
- moved C115 48.5 mm to (106.2, 65.5), turned to 180 degrees
- moved C113 47.6 mm to (110.1, 66.0), turned to 90 degrees
- moved C119 46.2 mm to (112.4, 64.3)
- moved C112 38.1 mm to (101.4, 68.8), turned to 180 degrees
- moved C111 35.2 mm to (101.4, 70.6), turned to 180 degrees
- moved R41 4.71 mm to (115.4, 37.7)
- moved C124 4.62 mm to (110.8, 73.9), turned to 180 degrees
- moved C126 2.28 mm to (110.8, 72.1), turned to 180 degrees
Connections:
- SW4 pad 1: /hdmitx1/AV2_AUD_R -> /hdmitx1/AV2_AUD_L
- SW4 pad 2: Net-(J6-Pad3) -> Net-(J6-Pad2)
- SW4 pad 3: /hdmitx1/AV1_AUD_R -> /hdmitx1/AV1_AUD_L
- SW4 pad 4: /hdmitx1/AV2_AUD_L -> /hdmitx1/AV2_AUD_R
- SW4 pad 5: Net-(J6-Pad2) -> Net-(J6-Pad3)
- SW4 pad 6: /hdmitx1/AV1_AUD_L -> /hdmitx1/AV1_AUD_R
Routing:
- net GND: track 1210.6 -> 1327.5 mm, vias 225 -> 240
- net /hdmitx1/AV3_AUD_R: track 0.00 -> 47.3 mm, vias 0 -> 1
- net /hdmitx1/AV3_AUD_L: track 0.00 -> 44.1 mm, vias 0 -> 2
- net /hdmitx1/AV1_AUD_L: track 0.47 -> 29.4 mm, vias 0 -> 2
- net /hdmitx1/AV1_AUD_R: track 0.33 -> 27.0 mm, vias 0 -> 2
- net /fpga1/SCL: track 201.9 -> 228.2 mm, vias 3 -> 5
- net /hdmitx1/HPD: track 8.15 -> 32.6 mm, vias 1 -> 2
- net /fpga1/SDA: track 190.3 -> 214.1 mm, vias 3 -> 5
- net /hdmitx1/AV2_AUD_L: track 0.00 -> 17.2 mm, vias 0 -> 2
- net /hdmitx1/AV2_AUD_R: track 0.00 -> 15.9 mm, vias 0 -> 2
- net Net-(J6-Pad2): track 0.45 -> 13.8 mm
- net Net-(J6-Pad3): track 0.00 -> 9.59 mm
- net /hdmitx1/5V: track 220.1 -> 229.4 mm, vias 0 -> 1
- net /hdmitx1/DVDD3V3: track 608.6 -> 614.8 mm, vias 31 -> 32
- net /hdmitx1/AVDD3V3: track 140.3 -> 145.7 mm, vias 8 -> 9
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
Commit message: v1.6-jp21
Parts:
- J3: value SCART-F -> JP21
Connections:
- J3 pad 1: Net-(J3-Pad1) -> /hdmitx1/AV1_AUD_L
- J3 pad 11: /tvp_board1/RGB1_G -> Net-(J3-Pad11)
- J3 pad 19: Net-(J3-Pad19) -> /tvp_board1/RGB1_G
- J3 pad 2: /hdmitx1/AV1_AUD_R -> Net-(J3-Pad2)
- J3 pad 20: /tvp_board1/RGB1_S -> /tvp_board1/RGB1_B
- J3 pad 3: Net-(J3-Pad3) -> GND
- J3 pad 5: GND -> /hdmitx1/AV1_AUD_R
- J3 pad 6: /hdmitx1/AV1_AUD_L -> Net-(J3-Pad6)
- J3 pad 7: /tvp_board1/RGB1_B -> GND
- J3 pad 8: Net-(J3-Pad8) -> GND
- J3 pad 9: GND -> /tvp_board1/RGB1_S
Routing:
- net /tvp_board1/RGB1_S: track 95.9 -> 124.5 mm
- net /tvp_board1/RGB1_G: track 46.3 -> 31.3 mm
- net /tvp_board1/RGB1_B: track 53.8 -> 63.0 mm
- net GND: track 1327.5 -> 1319.2 mm, vias 240 -> 239
- net /hdmitx1/AV1_AUD_R: track 27.0 -> 22.1 mm
- net /hdmitx1/AV1_AUD_L: track 29.4 -> 31.2 mm, vias 2 -> 3
Other:
- board text added: "OSSC v1.6-JP21"
- board text removed: "OSSC v1.6"
