File: fpga.sch (KiCad schematic (older format))
At the start: 83 parts, among them P1 JTAG_CONN, P3 mSD_CONN, Q1 BC847, Q2 BC857, SW2 SW_PUSH, SW3 SW_PUSH, U10 S25FL216K, U11 IRM-V538/TR1, U12 TLV70012, U13 TLV70025, U14 TLV70012, U2 EP4CE15E22

Commit message: - Update schematics and board to KiCAD 5.x
Parts:
- C101, C102, C108, C29, C30, C39, C40, C41, C42, C43, C44, C45, C46, C47, C48, C49, C50, C51, C52, C53, C54, C55, C56, C57, C58, C59, C60, C61, C62, C63, C64, C65, C66, C67, C68, C91, C92, C94, C96, C97, C98, C99: symbol C-RESCUE-ossc_board -> ossc_board-rescue:C-RESCUE-ossc_board
- D1, D2: symbol LED-RESCUE-ossc_board -> ossc_board-rescue:LED-RESCUE-ossc_board
- D3, D4: symbol ZENER -> ossc_board-rescue:ZENER
- DS1: symbol CONN_01X12 -> ossc_board-rescue:CONN_01X12
- P1: symbol CONN_02X05 -> ossc_board-rescue:CONN_02X05
- P3: symbol CONN_01X08 -> ossc_board-rescue:CONN_01X08
- Q1: symbol BC849 -> ossc_board-rescue:BC849
- Q2: symbol BC857 -> ossc_board-rescue:BC857
- R16, R17, R18, R19, R20, R21, R22, R23, R24, R28, R29, R30, R31, R32, R33, R34, R35, R36: symbol R-RESCUE-ossc_board -> ossc_board-rescue:R-RESCUE-ossc_board
- R27, R37, R39, R40, R42, R43: symbol R -> ossc_board-rescue:R
- SW2, SW3: symbol SW_PUSH -> ossc_board-rescue:SW_PUSH
- U10: symbol S25FL216K -> ossc_board-rescue:S25FL216K
- U11: symbol CONN_01X03 -> ossc_board-rescue:CONN_01X03
- U12, U13, U14: symbol TLV71209DBV-RESCUE-ossc_board -> ossc_board-rescue:TLV71209DBV-RESCUE-ossc_board
- U2: symbol EP4CE15E22 -> ossc_board-rescue:EP4CE15E22
Connections:
- wire segments 153 -> 168

Commit message: update to Kicad 5.x symbols
Parts:
- C101, C102, C108, C29, C30, C39, C40, C41, C42, C43, C44, C45, C46, C47, C48, C49, C50, C51, C52, C53, C54, C55, C56, C57, C58, C59, C60, C61, C62, C63, C64, C65, C66, C67, C68, C91, C92, C94, C96, C97, C98, C99: symbol ossc_board-rescue:C-RESCUE-ossc_board -> Device:C
- D1, D2: symbol ossc_board-rescue:LED-RESCUE-ossc_board -> Device:LED
- D3, D4: symbol ossc_board-rescue:ZENER -> Device:D_Zener
- DS1: symbol ossc_board-rescue:CONN_01X12 -> Connector_Generic:Conn_01x12
- P1: symbol ossc_board-rescue:CONN_02X05 -> Connector_Generic:Conn_02x05_Odd_Even
- P3: symbol ossc_board-rescue:CONN_01X08 -> Connector_Generic:Conn_01x08
- Q1: symbol ossc_board-rescue:BC849 -> Transistor_BJT:BC847
- Q2: symbol ossc_board-rescue:BC857 -> Transistor_BJT:BC857
- R16, R17, R18, R19, R20, R21, R22, R23, R24, R28, R29, R30, R31, R32, R33, R34, R35, R36: symbol ossc_board-rescue:R-RESCUE-ossc_board -> Device:R
- R27, R37, R39, R40, R42, R43: symbol ossc_board-rescue:R -> Device:R
- SW2, SW3: symbol ossc_board-rescue:SW_PUSH -> Switch:SW_Push
- U10: symbol ossc_board-rescue:S25FL216K -> custom_components:S25FL216K
- U11: symbol ossc_board-rescue:CONN_01X03 -> Connector_Generic:Conn_01x03
- U12, U14: symbol ossc_board-rescue:TLV71209DBV-RESCUE-ossc_board -> Regulator_Linear:TLV70012_SOT23-5
- U13: symbol ossc_board-rescue:TLV71209DBV-RESCUE-ossc_board -> Regulator_Linear:TLV70025_SOT23-5
- U2: symbol ossc_board-rescue:EP4CE15E22 -> custom_components:EP4CE15E22
Connections:
- wire segments 168 -> 189
Other:
- moved on the sheet: C102, C108, C39, C40, C41, C42, C43, C44, C45, C46, C48, C49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

Commit message: update to pcb v1.7
Parts:
- removed D3, D4: SD05-7, custom_components:SOD-323_Handsoldering, symbol Device:D_Zener
- added D3, D4: PESD3V3V4UW, Package_TO_SOT_SMD:SOT-665, symbol custom_components:PESD5V0V4UW
- Q1, Q2: footprint Housings_SOT-23_SOT-143_TSOT-6:SOT-23_Handsoldering -> Package_TO_SOT_SMD:SOT-23_Handsoldering
Connections:
- wire segments 189 -> 194
- no-connect marks 3 -> 5
Changed lines of the file:
@@
 U 1 1 54FE12DE
 P 7050 3950
-F 0 "R18" V 7130 3950 40  0000 C CNN
+F 0 "R18" V 7000 4100 40  0000 C CNN
 F 1 "10k" V 7057 3951 40  0000 C CNN
 F 2 "custom_components:SM0603_Resistor_libcms" V 6980 3950 30  0001 C CNN
@@
 	-1   0    0    1
 $EndComp
-Wire Wire Line
-	6550 1550 6900 1550
 Wire Wire Line
 	6400 1150 7000 1150
@@
 F 0 "Q1" H 9000 4225 50  0000 L CNN
 F 1 "BC847" H 9000 4150 50  0000 L CNN
-F 2 "Housings_SOT-23_SOT-143_TSOT-6:SOT-23_Handsoldering" H 9000 4075 50  0001 L CIN
+F 2 "Package_TO_SOT_SMD:SOT-23_Handsoldering" H 9000 4075 50  0001 L CIN
 F 3 "" H 8800 4150 50  0000 L CNN
 	1    8800 4150
@@
 F 0 "Q2" H 9100 3525 50  0000 L CNN
 F 1 "BC857" H 9100 3450 50  0000 L CNN
-F 2 "Housings_SOT-23_SOT-143_TSOT-6:SOT-23_Handsoldering" H 9100 3375 50  0001 L CIN
+F 2 "Package_TO_SOT_SMD:SOT-23_Handsoldering" H 9100 3375 50  0001 L CIN
 F 3 "" H 8900 3450 50  0000 L CNN
 	1    8900 3450
@@
 Text Label 7900 6250 0    60   ~ 0
 VCCIO
-$Comp
-L Device:D_Zener D4
-U 1 1 58C55E08
-P 6900 1700
-F 0 "D4" H 6900 1800 50  0000 C CNN
-F 1 "SD05-7" H 6900 1600 50  0000 C CNN
-F 2 "custom_components:SOD-323_Handsoldering" H 6900 1700 60  0001 C CNN
-F 3 "" H 6900 1700 60  0000 C CNN
-	1    6900 1700
-	0    1    1    0
-$EndComp
-$Comp
-L power:GND #PWR077
-U 1 1 58C55E0F
-P 6900 1850
-F 0 "#PWR077" H 6900 1850 30  0001 C CNN
-F 1 "GND" H 6900 1780 30  0001 C CNN
-F 2 "" H 6900 1850 60  0001 C CNN
-F 3 "" H 6900 1850 60  0000 C CNN
-	1    6900 1850
-	1    0    0    -1
-$EndComp
-$Comp
-L Device:D_Zener D3
-U 1 1 58C560B1
-P 6400 1300
-F 0 "D3" H 6400 1400 50  0000 C CNN
-F 1 "SD05-7" H 6400 1200 50  0000 C CNN
-F 2 "custom_components:SOD-323_Handsoldering" H 6400 1300 60  0001 C CNN
-F 3 "" H 6400 1300 60  0000 C CNN
-	1    6400 1300
-	0    1    1    0
-$EndComp
-$Comp
-L power:GND #PWR078
-U 1 1 58C561E6
-P 6400 1450
-F 0 "#PWR078" H 6400 1450 30  0001 C CNN
-F 1 "GND" H 6400 1380 30  0001 C CNN
-F 2 "" H 6400 1450 60  0001 C CNN
-F 3 "" H 6400 1450 60  0000 C CNN
-	1    6400 1450
-	1    0    0    -1
-$EndComp
-Connection ~ 6900 1550
 Wire Wire Line
 	8850 5800 8850 6600
@@
 Wire Wire Line
 	8850 5050 8850 5800
-Wire Wire Line
-	6900 1550 7000 1550
 Wire Wire Line
 	8850 5800 9450 5800
@@
 	0    -1   -1   0
 $EndComp
+Wire Wire Line
+	6550 1550 7000 1550
+$Comp
+L custom_components:PESD5V0V4UW D4
+U 1 1 611E53FE
+P 9150 2800
+F 0 "D4" V 8683 2800 50  0000 C CNN
+F 1 "PESD3V3V4UW" V 8774 2800 50  0000 C CNN
+F 2 "Package_TO_SOT_SMD:SOT-665" H 9850 2550 50  0001 C CNN
+F 3 "" V 9150 2800 50  0001 C CNN
+	1    9150 2800
+	0    1    1    0
+$EndComp
+$Comp
+L power:GND #PWR0132
+U 1 1 611EF7F7
+P 8950 2800
+F 0 "#PWR0132" H 8950 2800 30  0001 C CNN
+F 1 "GND" H 8950 2730 30  0001 C CNN
+F 2 "" H 8950 2800 60  0001 C CNN
+F 3 "" H 8950 2800 60  0000 C CNN
+	1    8950 2800
+	0    1    1    0
+$EndComp
+Wire Wire Line
+	9600 2600 9350 2600
+Wire Wire Line
+	9600 2700 9350 2700
+Wire Wire Line
+	9600 2800 9350 2800
+Wire Wire Line
+	9600 2900 9350 2900
+Text Label 9400 2700 0    60   ~ 0
+TCK
+Text Label 9400 2600 0    60   ~ 0
+TDI
+Text Label 9400 2800 0    60   ~ 0
+TDO
+Text Label 9400 2900 0    60   ~ 0
+TMS
+$Comp
+L power:GND #PWR078
+U 1 1 6126AEAE
+P 7550 950
+F 0 "#PWR078" H 7550 950 30  0001 C CNN
+F 1 "GND" H 7550 880 30  0001 C CNN
+F 2 "" H 7550 950 60  0001 C CNN
+F 3 "" H 7550 950 60  0000 C CNN
+	1    7550 950
+	0    1    1    0
+$EndComp
+Wire Wire Line
+	8250 750  7950 750
+Wire Wire Line
+	8250 850  7950 850
+$Comp
+L custom_components:PESD5V0V4UW D3
+U 1 1 61257495
+P 7750 950
+F 0 "D3" V 8000 950 50  0000 C CNN
+F 1 "PESD3V3V4UW" V 7374 950 50  0000 C CNN
+F 2 "Package_TO_SOT_SMD:SOT-665" H 8450 700 50  0001 C CNN
+F 3 "" V 7750 950 50  0001 C CNN
+	1    7750 950
+	0    1    1    0
+$EndComp
+NoConn ~ 7950 950
+NoConn ~ 7950 1050
+Text Label 8000 750  0    60   ~ 0
+BTN0
+Text Label 8000 850  0    60   ~ 0
+BTN1
 $EndSCHEMATC
