File: ossc_board.sch (KiCad schematic (older format))
At the start: 4 parts

Commit message: - Update schematics and board to KiCAD 5.x
Parts:
- MH1, MH2, MH3, MH4: symbol CONN_01X01 -> ossc_board-rescue:CONN_01X01
Changed lines of the file:
@@
-EESchema Schematic File Version 2
-LIBS:power
-LIBS:device
-LIBS:transistors
-LIBS:conn
-LIBS:linear
-LIBS:regul
-LIBS:74xx
-LIBS:cmos4000
-LIBS:adc-dac
-LIBS:memory
-LIBS:xilinx
-LIBS:microcontrollers
-LIBS:dsp
-LIBS:microchip
-LIBS:analog_switches
-LIBS:motorola
-LIBS:texas
-LIBS:intel
-LIBS:audio
-LIBS:interface
-LIBS:digital-audio
-LIBS:philips
-LIBS:display
-LIBS:cypress
-LIBS:siliconi
-LIBS:opto
-LIBS:atmel
-LIBS:contrib
-LIBS:valves
-LIBS:custom_components
+EESchema Schematic File Version 4
 LIBS:ossc_board-cache
-EELAYER 25 0
+EELAYER 26 0
 EELAYER END
 $Descr A4 11693 8268
@@
 $EndSheet
 $Comp
-L CONN_01X01 MH1
+L ossc_board-rescue:CONN_01X01 MH1
 U 1 1 55126368
 P 1250 950
@@
 $EndComp
 $Comp
-L CONN_01X01 MH3
+L ossc_board-rescue:CONN_01X01 MH3
 U 1 1 55129B56
 P 1350 6250
@@
 $EndComp
 $Comp
-L CONN_01X01 MH2
+L ossc_board-rescue:CONN_01X01 MH2
 U 1 1 5512C83E
 P 10450 1000
@@
 $EndComp
 $Comp
-L CONN_01X01 MH4
+L ossc_board-rescue:CONN_01X01 MH4
 U 1 1 5512E422
 P 10400 6200
@@
 	3050 4300 4150 4300
 Wire Wire Line
-	3050 4600 4650 4600
-Wire Wire Line
-	3050 4700 4650 4700
+	3050 4600 4350 4600
+Wire Wire Line
+	3050 4700 4500 4700
 Wire Wire Line
 	6750 1050 8350 1050
@@
 	6750 4050 8350 4050
 Wire Wire Line
-	6750 4300 8350 4300
+	6750 4300 6950 4300
 Wire Wire Line
 	6750 4400 8350 4400
@@
 	8950 5700 9550 5700
 Wire Wire Line
-	3050 5550 8350 5550
+	3050 5550 3800 5550
 Wire Wire Line
 	3050 5650 8350 5650
@@
 Wire Wire Line
 	3050 6600 8350 6600
+Wire Wire Line
+	4500 4700 4650 4700
+Wire Wire Line
+	4350 4600 4650 4600
+Wire Wire Line
+	6950 4300 8350 4300
+Wire Wire Line
+	3800 5550 8350 5550
 $EndSCHEMATC

Commit message: update to Kicad 5.x symbols
Parts:
- MH1, MH2, MH3, MH4: symbol ossc_board-rescue:CONN_01X01 -> Mechanical:MountingHole
Connections:
- no-connect marks 4 -> 0

Commit message: update to pcb v1.7
Other:
- note added: "max. 175mA drawn"
- note removed: "max. 543mA drawn"
Changed lines of the file:
@@
 max. 230mA drawn
 Text Notes 1900 5450 0    60   ~ 0
-max. 543mA drawn
+max. 175mA drawn
 $Sheet
 S 8350 950  1650 5900
